File: LrE-6.pb/LrE-6.sch (KiCad schematic (older format))
At the start: 123 parts, among them J1 USB_B_Micro, J2 SM06B-SRSS-TB, J3 Conn_02x03_Row_Letter_First, J4 Conn_02x01, Q1 BSS138, Q11 BSS138, Q12 BSS138, Q13 BSS138, Q14 BSS138, Q2 BSS138, Q3 BSS138, Q4 BSS138, Q5 BSS138, SW1 SW_Push_45deg, SW10 SW_Push_45deg, SW11 Rotary_Encoder_Switch, SW12 Rotary_Encoder_Switch, SW13 Rotary_Encoder_Switch, SW14 Rotary_Encoder_Switch, SW15 Rotary_Encoder_Switch, SW16 Rotary_Encoder_Switch, SW2 SW_Push_45deg, SW3 SW_Push_45deg, SW4 SW_Push_45deg, SW5 SW_Push_45deg, SW6 SW_Push_45deg, SW7 SW_Push_45deg, SW8 SW_Push_45deg, SW9 SW_Push_45deg, U1 STM32F072C8Tx, U2 ESP-WROOM-02, U3 AQM0802-FLW-GBW, U4 SPX3819M5-L3-3TR

Commit message: revise PB to R1.11
Parts:
- added R33: 10K, Resistor_SMD:R_0805_2012Metric, symbol Device:R
- added R34: 100, Resistor_SMD:R_0805_2012Metric, symbol Device:R
Connections:
- wire segments 433 -> 441
- no-connect marks 10 -> 9
Other:
- note added: "R1.11"
- note removed: "R1.1"
- moved on the sheet: C27, R30, R31, R32

Commit message: R2.0
Board Revision 2.0 & firmware working for board 2.0
Parts:
- removed D17: LED_RABG, LED_SMD:LED_Avago_PLCC4_3.2x2.8mm_CW, symbol Device:LED_RABG
- removed D20: LED RD, LED_SMD:LED_0805_2012Metric, symbol Device:LED
- removed D21, D22, D23, D24, D25: LED YW, LED_SMD:LED_0805_2012Metric, symbol Device:LED
- removed Q1, Q12, Q13, Q14, Q2, Q3, Q4, Q5: BSS138, Package_TO_SOT_SMD:SOT-23, symbol Transistor_FET:BSS138
- removed R22, R23: 100, Resistor_SMD:R_0805_2012Metric, symbol Device:R
- removed R25, R26, R27, R28, R29: 240, Resistor_SMD:R_0805_2012Metric, symbol Device:R
- removed R30: 10K, Resistor_SMD:R_0805_2012Metric, symbol Device:R
- removed R32: 150, Resistor_SMD:R_0805_2012Metric, symbol Device:R
- added C31, C32, C33, C34, C35, C36: 0.1u, Capacitor_SMD:C_0805_2012Metric, symbol Device:C
- added D31, D32, D33, D34, D35, D36: WS2812B, LrE-6:LED_WS2812B-2020, symbol LrE-6:WS2812B-2020
- added Q1: 2N7002, Package_TO_SOT_SMD:SOT-23, symbol Transistor_FET:2N7002
- C1, C10, C11, C12, C13, C14, C15, C16, C17, C18, C19, C2, C20, C21, C22, C23, C24, C25, C26, C27, C28, C3, C4, C5, C6, C7, C8, C9: symbol Device:C -> LrE-6-rescue:C-Device
- D1, D10, D11, D12, D13, D14, D15, D16, D2, D3, D4, D5, D6, D7, D8, D9: symbol Diode:1N4148W -> LrE-6-rescue:1N4148W-Diode
- D18: symbol Device:LED -> LrE-6-rescue:LED-Device
- D19: value LED OR -> LED BL; symbol Device:LED -> LrE-6-rescue:LED-Device
- H1, H2, H3, H4: symbol Mechanical:MountingHole -> LrE-6-rescue:MountingHole-Mechanical
- J1: symbol Connector:USB_B_Micro -> LrE-6-rescue:USB_B_Micro-Connector
- J2: symbol Connector_Generic:Conn_01x06 -> LrE-6-rescue:Conn_01x06-Connector_Generic
- J3: value Conn_02x03_Row_Letter_First -> LP_Header_02x03; symbol Connector_Generic:Conn_02x03_Odd_Even -> LrE-6-rescue:Conn_02x03_Odd_Even-Connector_Generic
- J4: value Conn_02x01 -> LP_Header_01x02; symbol Connector_Generic:Conn_02x01 -> LrE-6-rescue:Conn_02x01-Connector_Generic
- Q11: value BSS138 -> 2N7002; symbol Transistor_FET:BSS138 -> LrE-6-rescue:2N7002-Transistor_FET
- R1, R10, R11, R12, R13, R14, R15, R16, R17, R18, R19, R2, R20, R24, R3, R33, R34, R4, R5, R6, R7, R8, R9: symbol Device:R -> LrE-6-rescue:R-Device
- R21: value 100 -> 4.7K
- R31: value 150 -> 75; symbol Device:R -> LrE-6-rescue:R-Device
- SW1, SW10, SW2, SW3, SW4, SW5, SW6, SW7, SW8, SW9: symbol Switch:SW_Push_45deg -> LrE-6-rescue:SW_Push_45deg-Switch
- SW11, SW12, SW13, SW14, SW15, SW16: symbol Device:Rotary_Encoder_Switch -> LrE-6-rescue:Rotary_Encoder_Switch-Device
- TP1: symbol Connector:TestPoint -> LrE-6-rescue:TestPoint-Connector
- U1: symbol MCU_ST_STM32F0:STM32F072C8Tx -> LrE-6-rescue:STM32F072C8Tx-MCU_ST_STM32F0
- U2: symbol RF_Module:ESP-WROOM-02 -> LrE-6-rescue:ESP-WROOM-02-RF_Module
- U4: symbol Regulator_Linear:LDK130-08_SOT23_SOT353 -> LrE-6-rescue:LDK130-08_SOT23_SOT353-Regulator_Linear
Connections:
- net labels added: LED1OUT, LED2OUT, LED3OUT, LED4OUT, LED5OUT, LED_DON, LED_DOUT, WL_0, WL_EN, WL_RST
- net labels removed: CB, CG, CR, DB, DG, DR, IND1, IND2, IND3, IND4, IND5, LED_B, LED_G, LED_R, WL_LED4
- wire segments 441 -> 457
- no-connect marks 9 -> 15
Other:
- note added: "FT234X"
- note added: "R2.0"
- note removed: "FT234X\n(Reverse)"
- note removed: "R1.11"
- moved on the sheet: C10, C11, C12, C20, C21, C23, C28, C3, C4, C5, C6, C9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

Commit message: LrE6 Board R2.01
Parts:
- removed D19: LED BL, LED_SMD:LED_0805_2012Metric, symbol LrE-6-rescue:LED-Device
- removed R31: 75, Resistor_SMD:R_0805_2012Metric, symbol LrE-6-rescue:R-Device
- added C30: 0.1u, Capacitor_SMD:C_0805_2012Metric, symbol Device:C
- added R36, R37: 10K, Resistor_SMD:R_0805_2012Metric, symbol Device:R
- D1, D10, D11, D12, D13, D14, D15, D16, D2, D3, D4, D5, D6, D7, D8, D9: footprint Diode_SMD:D_SOD-123 -> LrE-6:D_SOD-123
- SW11, SW12, SW13, SW14, SW15, SW16: footprint Rotary_Encoder:RotaryEncoder_Alps_EC11E-Switch_Vertical_H20mm -> LrE-6:RotaryEncoder_EC11E-SMD
Connections:
- net labels removed: WL_LED5
- wire segments 457 -> 462
- no-connect marks 15 -> 19
Other:
- note added: "R2.01"
- note removed: "R2.0"

Commit message: 0.22-pre1
Other:
- note added: "R2.02"
- note removed: "R2.01"
Changed lines of the file:
@@
 	12250 4150 12700 4150
 Text Notes 15150 9550 0    197  ~ 0
-R2.01
+R2.02
 Wire Wire Line
 	11750 3250 12700 3250

Commit message: 0.24-pre5
Connections:
- net labels added: ENC0-A, ENC0-B
Changed lines of the file:
@@
 	7800 5050 7300 5050
 Text Label 7300 4950 0    50   ~ 0
-ENC6-A
+ENC0-A
 Text Label 7300 5050 0    50   ~ 0
-ENC6-B
+ENC0-B
 $Comp
 L LrE-6-rescue:Rotary_Encoder_Switch-Device SW11

Commit message: 0.27-5
Parts:
- removed C20: 0.1u, Capacitor_SMD:C_0805_2012Metric, symbol LrE-6-rescue:C-Device
- removed C28: 10u, Capacitor_SMD:C_0805_2012Metric, symbol LrE-6-rescue:C-Device
- removed J3: LP_Header_02x03, Connector_PinHeader_2.54mm:PinHeader_2x03_P2.54mm_Vertical, symbol LrE-6-rescue:Conn_02x03_Odd_Even-Connector_Generic
- removed J4: LP_Header_01x02, Connector_PinHeader_2.54mm:PinHeader_1x02_P2.54mm_Vertical, symbol LrE-6-rescue:Conn_02x01-Connector_Generic
- removed R33: 10K, Resistor_SMD:R_0805_2012Metric, symbol LrE-6-rescue:R-Device
- removed R34: 100, Resistor_SMD:R_0805_2012Metric, symbol LrE-6-rescue:R-Device
- removed R36, R37: 10K, Resistor_SMD:R_0805_2012Metric, symbol Device:R
- removed U2: ESP-WROOM-02, RF_Module:ESP-WROOM-02, symbol LrE-6-rescue:ESP-WROOM-02-RF_Module
- C30, C31, C32, C33, C34, C35, C36: symbol Device:C -> LrE-6-rescue:C-Device
- Q1: symbol Transistor_FET:2N7002 -> LrE-6-rescue:2N7002-Transistor_FET
- R21: symbol Device:R -> LrE-6-rescue:R-Device
Connections:
- net labels removed: ENC6-A, ENC6-B, STM_RX, STM_TX, WL_0, WL_EN, WL_RST, WL_RXD, WL_TXD
- wire segments 462 -> 419
- no-connect marks 19 -> 14
Other:
- note added: "R2.1\n"
- note removed: "FT234X"
- note removed: "GND"
- note removed: "N.C.(5V)"
- note removed: "R2.02"
- note removed: "RXD"
- note removed: "TXD"
- moved on the sheet: Q1, R21

Commit message: pb R2.1pre
Parts:
- removed Q11: 2N7002, Package_TO_SOT_SMD:SOT-23, symbol LrE-6-rescue:2N7002-Transistor_FET
- removed U3: AQM0802-FLW-GBW, LrE-6:AQM0802_1, symbol LrE-6-rescue:AQM-LrE-6
- added C20: 1u, Capacitor_SMD:C_0805_2012Metric, symbol LrE-6-rescue:C-Device
- added C28, C29: 2.2u, Capacitor_SMD:C_0805_2012Metric, symbol LrE-6-rescue:C-Device
- added TP2, TP3: TestPoint-Connector, TestPoint:TestPoint_THTPad_D2.0mm_Drill1.0mm, symbol LrE-6-rescue:TestPoint-Connector
- added U3: OLED-0.91, LrE-6:OLED-9.1, symbol LrE-6:OLED-0.91
- C23, C24: footprint Capacitor_SMD:C_0603_1608Metric -> Capacitor_SMD:C_0805_2012Metric
- C27: value 0.1u -> 1u; footprint Capacitor_SMD:C_0603_1608Metric -> Capacitor_SMD:C_0805_2012Metric
- R18: value 10 -> 390K
- R19, R20: footprint Resistor_SMD:R_0805_2012Metric -> Resistor_SMD:R_0603_1608Metric
Connections:
- net labels removed: BL_A, BL_K, BL_ON
- wire segments 419 -> 429
Other:
- moved on the sheet: C21, C23, C24, C27, J2, Q1, R17, R18, R19, R20, R21

Commit message: 0.28-3
Other:
- note added: "R2.2\n"
- note removed: "R2.1\n"
Changed lines of the file:
@@
 	11650 1700 11650 1650
 Text Notes 15300 9850 0    197  ~ 0
-R2.1\n
+R2.2\n
 Wire Wire Line
 	1200 10900 1700 10900
