File: LrE-6.pb/LrE-6.sch (KiCad schematic (older format))
At the start: 110 parts, among them J1 USB_B_Micro, J2 SM06B-SRSS-TB, Q1 2N7002, SW1 Tact_SW_8mm, SW10 Tact_SW_8mm, SW11 EC11_SMD, SW12 EC11_SMD, SW13 EC11_SMD, SW14 EC11_SMD, SW15 EC11_SMD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

Commit message: First commit for F3.2PB
Parts:
- SW11, SW12, SW13, SW14, SW15, SW16: footprint LrE-6:RotaryEncoder_EC11E-SMD2 -> Rotary_Encoder:RotaryEncoder_Alps_EC11E-Switch_Vertical_H20mm
Changed lines of the file:
@@
 F 0 "SW11" H 2300 1817 50  0000 C CNN
 F 1 "EC11_SMD" H 2300 1726 50  0000 C CNN
-F 2 "LrE-6:RotaryEncoder_EC11E-SMD2" H 2150 1610 50  0001 C CNN
+F 2 "Rotary_Encoder:RotaryEncoder_Alps_EC11E-Switch_Vertical_H20mm" H 2150 1610 50  0001 C CNN
 F 3 "~" H 2300 1710 50  0001 C CNN
 	1    2300 1450
@@
 F 0 "SW12" H 2350 3467 50  0000 C CNN
 F 1 "EC11_SMD" H 2350 3376 50  0000 C CNN
-F 2 "LrE-6:RotaryEncoder_EC11E-SMD2" H 2200 3260 50  0001 C CNN
+F 2 "Rotary_Encoder:RotaryEncoder_Alps_EC11E-Switch_Vertical_H20mm" H 2200 3260 50  0001 C CNN
 F 3 "~" H 2350 3360 50  0001 C CNN
 	1    2350 3100
@@
 F 0 "SW13" H 2450 5217 50  0000 C CNN
 F 1 "EC11_SMD" H 2450 5126 50  0000 C CNN
-F 2 "LrE-6:RotaryEncoder_EC11E-SMD2" H 2300 5010 50  0001 C CNN
+F 2 "Rotary_Encoder:RotaryEncoder_Alps_EC11E-Switch_Vertical_H20mm" H 2300 5010 50  0001 C CNN
 F 3 "~" H 2450 5110 50  0001 C CNN
 	1    2450 4850
@@
 F 0 "SW14" H 5000 1767 50  0000 C CNN
 F 1 "EC11_SMD" H 5000 1676 50  0000 C CNN
-F 2 "LrE-6:RotaryEncoder_EC11E-SMD2" H 4850 1560 50  0001 C CNN
+F 2 "Rotary_Encoder:RotaryEncoder_Alps_EC11E-Switch_Vertical_H20mm" H 4850 1560 50  0001 C CNN
 F 3 "~" H 5000 1660 50  0001 C CNN
 	1    5000 1400
@@
 F 0 "SW15" H 5150 3467 50  0000 C CNN
 F 1 "EC11_SMD" H 5150 3376 50  0000 C CNN
-F 2 "LrE-6:RotaryEncoder_EC11E-SMD2" H 5000 3260 50  0001 C CNN
+F 2 "Rotary_Encoder:RotaryEncoder_Alps_EC11E-Switch_Vertical_H20mm" H 5000 3260 50  0001 C CNN
 F 3 "~" H 5150 3360 50  0001 C CNN
 	1    5150 3100
@@
 F 0 "SW16" H 5250 5217 50  0000 C CNN
 F 1 "EC11_SMD" H 5250 5126 50  0000 C CNN
-F 2 "LrE-6:RotaryEncoder_EC11E-SMD2" H 5100 5010 50  0001 C CNN
+F 2 "Rotary_Encoder:RotaryEncoder_Alps_EC11E-Switch_Vertical_H20mm" H 5100 5010 50  0001 C CNN
 F 3 "~" H 5250 5110 50  0001 C CNN
 	1    5250 4850
