File: LrE-6.pb/LrE-6.kicad_pcb (KiCad board)
At the start: 2 copper layers, 100 x 100 mm, 117 parts, among them J1 USB_B_Micro, J2 SM06B-SRSS-TB, J3 LP_Header_02x03, J4 LP_Header_01x02, Q1 2N7002, Q11 2N7002, SW1 SW_Push_45deg, SW10 SW_Push_45deg, SW11 Rotary_Encoder_Switch, SW12 Rotary_Encoder_Switch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

Commit message: 0.22-pre1
Routing:
- net /LED1OUT: track 36.0 -> 35.4 mm
Other:
- board text added: "R2.02"
- board text removed: "R2.01"

Commit message: 0.22
Other:
- board text added: "Scene"
- board text removed: "Mode"
Changed lines of the file:
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@@
-(kicad_pcb (version 20171130) (host pcbnew "(5.1.2)-1")
+(kicad_pcb (version 20171130) (host pcbnew "(5.1.2)-2")
   (general
     (thickness 1.2)
@@
     (effects (font (size 0.8 0.8) (thickness 0.15)))
   )
-  (gr_line (start 154.8 146.6) (end 148.4 146.6) (layer F.SilkS) (width 0.2))
-  (gr_line (start 154.8 149.2) (end 154.8 146.6) (layer F.SilkS) (width 0.2))
-  (gr_line (start 148.4 149.2) (end 154.8 149.2) (layer F.SilkS) (width 0.2))
-  (gr_line (start 148.4 146.6) (end 148.4 149.2) (layer F.SilkS) (width 0.2))
-  (gr_text "Mode\n" (at 151.52 147.95) (layer F.SilkS)
+  (gr_line (start 155 146.6) (end 148 146.6) (layer F.SilkS) (width 0.2))
+  (gr_line (start 155 149.2) (end 155 146.6) (layer F.SilkS) (width 0.2))
+  (gr_line (start 148 149.2) (end 155 149.2) (layer F.SilkS) (width 0.2))
+  (gr_line (start 148 146.6) (end 148 149.2) (layer F.SilkS) (width 0.2))
+  (gr_text Scene (at 151.52 147.95) (layer F.SilkS)
     (effects (font (size 1.5 1.5) (thickness 0.2)))
   )

Commit message: 0.23-pre
Other:
- board text removed: "Select"
Changed lines of the file:
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@@
   (general
     (thickness 1.2)
-    (drawings 55)
+    (drawings 50)
     (tracks 1335)
     (zones 0)
@@
       (xy -8.140177 0.656392)) (layer B.SilkS) (width 0.01))
   )
-  (gr_line (start 85.61 123.8) (end 79 123.8) (layer F.SilkS) (width 0.15))
-  (gr_line (start 85.7 126) (end 85.7 123.84) (layer F.SilkS) (width 0.15))
-  (gr_line (start 79 126) (end 85.7 126) (layer F.SilkS) (width 0.15))
-  (gr_line (start 79 123.91) (end 79 125.92) (layer F.SilkS) (width 0.15))
-  (gr_text Select (at 82.32 124.84) (layer F.SilkS)
-    (effects (font (size 1.2 1.2) (thickness 0.2)))
-  )
   (gr_text GND (at 159.09 87.5) (layer F.SilkS)

Commit message: 0.24-pre5
Connections:
- net /ENC6-A renamed /ENC0-A
- net /ENC6-B renamed /ENC0-B
Other:
- board text added: "0"
- board text added: "1"
- board text added: "2"
- board text added: "3"
- board text added: "4"
- board text added: "5"
- board text added: "6"
- board text added: "7"
- board text added: "8"

Commit message: 0.27-5
Parts:
- removed C20: 0.1u, Capacitor_SMD:C_0805_2012Metric
- removed C28: 10u, Capacitor_SMD:C_0805_2012Metric
- removed J3: LP_Header_02x03, Connector_PinHeader_2.54mm:PinHeader_2x03_P2.54mm_Vertical
- removed J4: LP_Header_01x02, Connector_PinHeader_2.54mm:PinHeader_1x02_P2.54mm_Vertical
- removed R33, R36, R37: 10K, Resistor_SMD:R_0805_2012Metric
- removed R34: 100, Resistor_SMD:R_0805_2012Metric
- removed U2: ESP-WROOM-02, RF_Module:ESP-WROOM-02
- moved C26 3.00 mm to (119.4, 67.8)
- moved C25 2.83 mm to (111.8, 67.8)
- moved C30 1.39 mm to (159.7, 79.7)
Connections:
- D36 pad 1: Net-(D36-Pad1) -> (no net)
- J1 pad 4: Net-(J1-Pad4) -> (no net)
- J2 pad 6: Net-(J2-Pad6) -> (no net)
- U1 pad 17: Net-(U1-Pad17) -> (no net)
- U1 pad 18: Net-(U1-Pad18) -> (no net)
- U1 pad 19: Net-(U1-Pad19) -> (no net)
- U1 pad 2: Net-(U1-Pad2) -> (no net)
- U1 pad 27: Net-(U1-Pad27) -> (no net)
- U1 pad 28: Net-(U1-Pad28) -> (no net)
- U1 pad 29: /WL_RST -> (no net)
- U1 pad 30: /STM_TX -> (no net)
- U1 pad 31: /STM_RX -> (no net)
- U3 pad 1: Net-(U3-Pad1) -> (no net)
Routing:
- net /STM_TX: track 84.6 -> 0.00 mm
- net /STM_RX: track 81.4 -> 0.00 mm, vias 2 -> 0
- net /WL_RST: track 62.6 -> 0.00 mm, vias 4 -> 0
- net GND: track 159.2 -> 103.3 mm, vias 20 -> 18
- net +3V3: track 451.2 -> 433.4 mm
- net /WL_RXD: track 15.8 -> 0.00 mm
- net /WL_TXD: track 10.7 -> 0.00 mm
- net /WL_0: track 9.22 -> 0.00 mm, vias 1 -> 0
- net /VBUS: track 268.0 -> 262.0 mm
- net /WL_EN: track 5.40 -> 0.00 mm
- net Net-(R34-Pad1): track 2.58 -> 0.00 mm, vias 1 -> 0
Other:
- board text added: "R2.1"
- board text removed: "R2.02"
- board text removed: "RX"
- board text removed: "STM32"
- board text removed: "TX"
- board text removed: "UART DL"
- board text removed: "WROOM"

Commit message: pb R2.1pre
Parts:
- removed Q11: 2N7002, Package_TO_SOT_SMD:SOT-23
- added C20: 1u, Capacitor_SMD:C_0805_2012Metric, B.Cu at (140.3, 77.0)
- added C28: 2.2u, Capacitor_SMD:C_0805_2012Metric, B.Cu at (148.4, 66.5)
- added C29: 2.2u, Capacitor_SMD:C_0805_2012Metric, B.Cu at (150.4, 66.4)
- added TP2: TestPoint-Connector, TestPoint:TestPoint_THTPad_D2.0mm_Drill1.0mm, F.Cu at (125.0, 69.5)
- added TP3: TestPoint-Connector, TestPoint:TestPoint_THTPad_D2.0mm_Drill1.0mm, F.Cu at (125.0, 74.2)
- C23, C24: footprint Capacitor_SMD:C_0603_1608Metric -> Capacitor_SMD:C_0805_2012Metric
- C27: value 0.1u -> 1u; footprint Capacitor_SMD:C_0603_1608Metric -> Capacitor_SMD:C_0805_2012Metric
- R18: value 10 -> 390K
- R19, R20: moved to F.Cu
- TP1: value TestPoint -> TestPoint-Connector; footprint TestPoint:TestPoint_THTPad_D1.5mm_Drill0.7mm -> TestPoint:TestPoint_THTPad_D2.0mm_Drill1.0mm
- U3: value AQM0802-FLW-GBW -> OLED-0.91; footprint LrE-6:AQM0802_1 -> LrE-6:OLED-9.1
- moved R18 65.3 mm to (142.8, 66.5), turned to 90 degrees
- moved C24 64.2 mm to (149.5, 81.3), turned to 180 degrees
- moved C23 57.6 mm to (145.3, 81.2)
- moved R20 51.2 mm to (140.5, 66.7), turned to 270 degrees
- moved C27 50.0 mm to (140.3, 75.0), turned to 0 degrees
- moved R19 48.2 mm to (138.8, 66.7), turned to 270 degrees
- moved U3 40.8 mm to (128.3, 68.5)
- moved TP1 35.4 mm to (130.4, 61.1)
- moved C30 8.70 mm to (161.7, 88.2), turned to 180 degrees
- moved D18 2.53 mm to (123.0, 57.5)
- moved C26 1.40 mm to (118.4, 66.9), turned to 90 degrees
Connections:
- C24 pad 1: +3V3 -> Net-(C24-Pad1)
- C27 pad 1: +3V3 -> GND
- C27 pad 2: GND -> +3V3
- D36 pad 1: (no net) -> Net-(D36-Pad1)
- J1 pad 4: (no net) -> Net-(J1-Pad4)
- J2 pad 6: (no net) -> Net-(J2-Pad6)
- R18 pad 1: /BL_A -> Net-(R18-Pad1)
- R18 pad 2: +3V3 -> GND
- U1 pad 17: (no net) -> Net-(U1-Pad17)
- U1 pad 18: (no net) -> Net-(U1-Pad18)
- U1 pad 19: (no net) -> Net-(U1-Pad19)
- U1 pad 2: (no net) -> Net-(U1-Pad2)
- U1 pad 27: (no net) -> Net-(U1-Pad27)
- U1 pad 28: (no net) -> Net-(U1-Pad28)
- U1 pad 29: (no net) -> Net-(U1-Pad29)
- U1 pad 30: (no net) -> Net-(U1-Pad30)
- U1 pad 31: (no net) -> Net-(U1-Pad31)
- U1 pad 38: /BL_ON -> Net-(U1-Pad38)
- U3 pad 1: (no net) -> Net-(C23-Pad2)
- U3 pad 10: /BL_A -> GND
- U3 pad 11: /BL_K -> /SCL
- U3 pad 2: Net-(C24-Pad2) -> Net-(C23-Pad1)
- U3 pad 3: Net-(C23-Pad2) -> Net-(C24-Pad2)
- U3 pad 4: Net-(C23-Pad1) -> Net-(C24-Pad1)
- U3 pad 7: /SDA -> +3V3
- U3 pad 8: /SCL -> GND
- U3 pad 9: +3V3 -> /NRST
Routing:
- net /NRST: track 30.3 -> 99.5 mm, vias 4 -> 5
- net /SDA: track 13.8 -> 73.8 mm, vias 0 -> 3
- net /SCL: track 14.2 -> 72.8 mm, vias 0 -> 3
- net /BL_ON: track 15.1 -> 0.00 mm, vias 2 -> 0
- net +3V3: track 433.4 -> 423.1 mm, vias 16 -> 17
- net /L0: track 112.5 -> 121.9 mm
- net Net-(C24-Pad1): track 0.00 -> 9.33 mm
- net Net-(C29-Pad2): track 0.00 -> 7.56 mm
- net GND: track 103.3 -> 96.1 mm, vias 18 -> 20
- net /L2: track 152.8 -> 159.8 mm
- net /ENC3-A: track 98.9 -> 92.1 mm
- net Net-(R18-Pad1): track 0.00 -> 5.93 mm
- net Net-(C23-Pad1): track 2.34 -> 7.94 mm
- net Net-(C28-Pad2): track 0.00 -> 5.21 mm
- net Net-(C23-Pad2): track 2.44 -> 7.50 mm
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Other:
- outline, holes or cut-outs redrawn
- board text added: "SCL"
- board text added: "SDA"

Commit message: 0.28-3
Other:
- board text added: "R2.2"
- board text removed: "R2.1"
Changed lines of the file:
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@@
     (effects (font (size 1 1) (thickness 0.15)))
   )
-  (gr_text R2.1 (at 130 151.5) (layer F.SilkS)
+  (gr_text R2.2 (at 130 151.5) (layer F.SilkS)
     (effects (font (size 2.5 2) (thickness 0.3)))
   )

Commit message: 0.28-5
Parts:
- moved TP2 9.25 mm to (116.0, 71.7)
- moved TP3 6.83 mm to (118.2, 73.7)
Routing:
- net /SDA: track 73.8 -> 71.4 mm
- net /SCL: track 72.8 -> 71.7 mm
- net /L2: track 159.8 -> 159.1 mm
- net /ENC5-B: track 110.8 -> 110.2 mm
- net /ENC0-B: track 110.8 -> 111.4 mm
Other:
- board text added: "F2.2"
- board text removed: "R2.2"
