File: LrE-6.panel/LrE-6_panel.kicad_pcb (KiCad board)
At the start: 2 copper layers, 0 parts

Commit message: 0.28-4
Other:
- board text removed: "4xR2.0"
Changed lines of the file:
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@@
-(kicad_pcb (version 20171130) (host pcbnew "(5.1.2)-1")
+(kicad_pcb (version 20171130) (host pcbnew "(5.0.2)-1")
   (general
     (thickness 1.6)
-    (drawings 105)
+    (drawings 98)
     (tracks 0)
     (zones 0)
@@
     (zone_45_only no)
     (trace_min 0.2)
+    (segment_width 0.2)
+    (edge_width 0.15)
     (via_size 0.8)
     (via_drill 0.4)
@@
     (uvia_min_size 0.2)
     (uvia_min_drill 0.1)
-    (edge_width 0.15)
-    (segment_width 0.2)
     (pcb_text_width 0.3)
     (pcb_text_size 1.5 1.5)
@@
     (uvia_drill 0.1)
   )
-  (gr_text 4xR2.0 (at 38.3286 40.5638) (layer Dwgs.User)
-    (effects (font (size 1.5 1.5) (thickness 0.3)))
-  )
-  (gr_line (start 41.8084 41.8084) (end 50.1904 50.2158) (layer Dwgs.User) (width 0.15))
-  (gr_line (start 34.3154 41.8592) (end 41.8592 41.8592) (layer Dwgs.User) (width 0.15))
-  (gr_arc (start 51.943001 51.968399) (end 51.9938 49.9364) (angle -90) (layer Dwgs.User) (width 0.2))
-  (gr_arc (start 147.980401 52.070001) (end 150.0124 52.1208) (angle -90) (layer Dwgs.User) (width 0.2))
-  (gr_arc (start 147.980399 147.955001) (end 147.9296 149.987) (angle -90) (layer Dwgs.User) (width 0.2))
-  (gr_arc (start 52.069999 147.954999) (end 50.038 147.9042) (angle -90) (layer Dwgs.User) (width 0.2))
   (gr_text 15 (at 130.6 158.3) (layer Dwgs.User)
     (effects (font (size 1.5 1.5) (thickness 0.3)))
@@
   (gr_circle (center 145 55) (end 146.523155 55) (layer Dwgs.User) (width 0.2))
   (gr_circle (center 55 55) (end 56.6 55) (layer Dwgs.User) (width 0.2))
-  (gr_line (start 50 52) (end 50 148) (layer Dwgs.User) (width 0.2))
-  (gr_line (start 52 150) (end 148 150) (layer Dwgs.User) (width 0.2))
-  (gr_line (start 150 52) (end 150 148) (layer Dwgs.User) (width 0.2))
-  (gr_line (start 52 50) (end 148 50) (layer Dwgs.User) (width 0.2))
+  (gr_line (start 50 50) (end 50 150) (layer Dwgs.User) (width 0.2))
+  (gr_line (start 50 150) (end 150 150) (layer Dwgs.User) (width 0.2))
+  (gr_line (start 150 50) (end 150 150) (layer Dwgs.User) (width 0.2))
+  (gr_line (start 50 50) (end 150 50) (layer Dwgs.User) (width 0.2))
 )

Commit message: 0.28-5
Other:
- board text added: "4xR2.0"
- board text added: "F2.2"
Changed lines of the file:
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@@
-(kicad_pcb (version 20171130) (host pcbnew "(5.0.2)-1")
+(kicad_pcb (version 20171130) (host pcbnew "(5.1.5)-3")
   (general
     (thickness 1.6)
-    (drawings 98)
+    (drawings 106)
     (tracks 0)
     (zones 0)
@@
     (zone_45_only no)
     (trace_min 0.2)
-    (segment_width 0.2)
-    (edge_width 0.15)
     (via_size 0.8)
     (via_drill 0.4)
@@
     (uvia_min_size 0.2)
     (uvia_min_drill 0.1)
+    (edge_width 0.15)
+    (segment_width 0.2)
     (pcb_text_width 0.3)
     (pcb_text_size 1.5 1.5)
@@
     (uvia_drill 0.1)
   )
+  (gr_text F2.2 (at 204.41412 173.609) (layer Dwgs.User)
+    (effects (font (size 3 3) (thickness 0.3)))
+  )
+  (gr_text 4xR2.0 (at 38.3286 40.5638) (layer Dwgs.User)
+    (effects (font (size 1.5 1.5) (thickness 0.3)))
+  )
+  (gr_line (start 41.8084 41.8084) (end 50.1904 50.2158) (layer Dwgs.User) (width 0.15))
+  (gr_line (start 34.3154 41.8592) (end 41.8592 41.8592) (layer Dwgs.User) (width 0.15))
+  (gr_arc (start 51.943001 51.968399) (end 51.9938 49.9364) (angle -90) (layer Dwgs.User) (width 0.2))
+  (gr_arc (start 147.980401 52.070001) (end 150.0124 52.1208) (angle -90) (layer Dwgs.User) (width 0.2))
+  (gr_arc (start 147.980399 147.955001) (end 147.9296 149.987) (angle -90) (layer Dwgs.User) (width 0.2))
+  (gr_arc (start 52.069999 147.954999) (end 50.038 147.9042) (angle -90) (layer Dwgs.User) (width 0.2))
   (gr_text 15 (at 130.6 158.3) (layer Dwgs.User)
     (effects (font (size 1.5 1.5) (thickness 0.3)))
@@
   (gr_circle (center 145 55) (end 146.523155 55) (layer Dwgs.User) (width 0.2))
   (gr_circle (center 55 55) (end 56.6 55) (layer Dwgs.User) (width 0.2))
-  (gr_line (start 50 50) (end 50 150) (layer Dwgs.User) (width 0.2))
-  (gr_line (start 50 150) (end 150 150) (layer Dwgs.User) (width 0.2))
-  (gr_line (start 150 50) (end 150 150) (layer Dwgs.User) (width 0.2))
-  (gr_line (start 50 50) (end 150 50) (layer Dwgs.User) (width 0.2))
+  (gr_line (start 50 52) (end 50 148) (layer Dwgs.User) (width 0.2))
+  (gr_line (start 52 150) (end 148 150) (layer Dwgs.User) (width 0.2))
+  (gr_line (start 150 52) (end 150 148) (layer Dwgs.User) (width 0.2))
+  (gr_line (start 52 50) (end 148 50) (layer Dwgs.User) (width 0.2))
 )
