File: LrE-6.4lpb/LrE-6.kicad_pcb (KiCad board)
At the start: 2 copper layers, 100 x 100 mm, 112 parts, among them J1 USB_B_Micro, J2 SM06B-SRSS-TB, Q1 2N7002, SW1 Tact_SW_8mm, SW10 Tact_SW_8mm, SW11 EC11_SMD, SW12 EC11_SMD, SW13 EC11_SMD, SW14 EC11_SMD, SW15 EC11_SMD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

Commit message: F4.0 board order
Parts:
- moved C16 2.77 mm to (120.8, 119.5), turned to 0 degrees
- moved C30 0.68 mm to (196.0, 133.2)
- moved D36 0.50 mm to (190.0, 160.5)
- moved C36 0.39 mm to (189.8, 162.7)
- moved C33 0.29 mm to (129.8, 162.8)
- moved C34 0.18 mm to (149.8, 162.8)
- moved C32 0.15 mm to (109.8, 162.8)
- moved C35 0.12 mm to (169.8, 162.8)
Routing:
- net +3V3: track 407.7 -> 70.8 mm, vias 18 -> 23
- net /VBUS: track 267.8 -> 33.1 mm, vias 2 -> 9
- net GND: track 136.7 -> 89.9 mm, vias 66 -> 65
- net /ENC0-A: track 136.7 -> 127.7 mm, vias 3 -> 2
- net /ENC3-B: track 72.7 -> 75.2 mm, vias 3 -> 2
- net /ENC1-A: track 72.1 -> 69.9 mm, vias 1 -> 0
- net /ENC4-A: track 92.1 -> 90.7 mm, vias 5 -> 4
- net /L3: track 130.3 -> 131.4 mm
- net /ENC2-A: track 45.8 -> 44.8 mm, vias 1 -> 0
- net /ENC4-B: track 85.3 -> 86.1 mm, vias 3 -> 2
- net /NRST: track 97.1 -> 96.4 mm, vias 5 -> 3
- net /LED1OUT: track 38.1 -> 37.4 mm
- net /ENC2-B: track 56.2 -> 55.6 mm, vias 3 -> 2
- net /ENC3-A: track 94.5 -> 95.0 mm
- net /SWDIO: track 18.2 -> 18.7 mm
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- added copper zone on In1.Cu, net +3V3
- added copper zone on In1.Cu, net /VBUS
- added copper zone on In2.Cu, net GND
Other:
- copper layers 2 -> 4
- board text added: "F4.0"
- board text removed: "-2"
- board text removed: "F2.8"
