File: LrE-6.2lpb/LrE-6.sch (KiCad schematic (older format))
At the start: 110 parts, among them J1 USB_B_Micro, J2 SM06B-SRSS-TB, Q1 2N7002, SW1 Tact_SW_8mm, SW10 Tact_SW_8mm, SW11 EC11_SMD, SW12 EC11_SMD, SW13 EC11_SMD, SW14 EC11_SMD, SW15 EC11_SMD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

Commit message: 0.45-2
Parts:
- C1, C10, C11, C12, C2, C3, C4, C5, C6, C7, C8, C9: value 0.01u -> 22n
- C25: value 0.01u -> 10n
Changed lines of the file:
@@
 P 1250 1750
 F 0 "C1" H 1365 1796 50  0000 L CNN
-F 1 "0.01u" H 1300 1650 50  0000 L CNN
+F 1 "22n" H 1300 1650 50  0000 L CNN
 F 2 "Capacitor_SMD:C_0805_2012Metric" H 1288 1600 50  0001 C CNN
 F 3 "~" H 1250 1750 50  0001 C CNN
@@
 P 1600 1750
 F 0 "C2" H 1715 1796 50  0000 L CNN
-F 1 "0.01u" H 1650 1650 50  0000 L CNN
+F 1 "22n" H 1650 1650 50  0000 L CNN
 F 2 "Capacitor_SMD:C_0805_2012Metric" H 1638 1600 50  0001 C CNN
 F 3 "~" H 1600 1750 50  0001 C CNN
@@
 P 1350 3400
 F 0 "C3" H 1465 3446 50  0000 L CNN
-F 1 "0.01u" H 1400 3300 50  0000 L CNN
+F 1 "22n" H 1400 3300 50  0000 L CNN
 F 2 "Capacitor_SMD:C_0805_2012Metric" H 1388 3250 50  0001 C CNN
 F 3 "~" H 1350 3400 50  0001 C CNN
@@
 P 1700 3400
 F 0 "C4" H 1815 3446 50  0000 L CNN
-F 1 "0.01u" H 1750 3300 50  0000 L CNN
+F 1 "22n" H 1750 3300 50  0000 L CNN
 F 2 "Capacitor_SMD:C_0805_2012Metric" H 1738 3250 50  0001 C CNN
 F 3 "~" H 1700 3400 50  0001 C CNN
@@
 P 4000 1750
 F 0 "C7" H 4115 1796 50  0000 L CNN
-F 1 "0.01u" H 4050 1650 50  0000 L CNN
+F 1 "22n" H 4050 1650 50  0000 L CNN
 F 2 "Capacitor_SMD:C_0805_2012Metric" H 4038 1600 50  0001 C CNN
 F 3 "~" H 4000 1750 50  0001 C CNN
@@
 P 4350 1750
 F 0 "C8" H 4465 1796 50  0000 L CNN
-F 1 "0.01u" H 4400 1650 50  0000 L CNN
+F 1 "22n" H 4400 1650 50  0000 L CNN
 F 2 "Capacitor_SMD:C_0805_2012Metric" H 4388 1600 50  0001 C CNN
 F 3 "~" H 4350 1750 50  0001 C CNN
@@
 P 4100 3450
 F 0 "C9" H 4215 3496 50  0000 L CNN
-F 1 "0.01u" H 4150 3350 50  0000 L CNN
+F 1 "22n" H 4150 3350 50  0000 L CNN
 F 2 "Capacitor_SMD:C_0805_2012Metric" H 4138 3300 50  0001 C CNN
 F 3 "~" H 4100 3450 50  0001 C CNN
@@
 P 4450 3450
 F 0 "C10" H 4565 3496 50  0000 L CNN
-F 1 "0.01u" H 4500 3350 50  0000 L CNN
+F 1 "22n" H 4500 3350 50  0000 L CNN
 F 2 "Capacitor_SMD:C_0805_2012Metric" H 4488 3300 50  0001 C CNN
 F 3 "~" H 4450 3450 50  0001 C CNN
@@
 P 4200 5150
 F 0 "C11" H 4315 5196 50  0000 L CNN
-F 1 "0.01u" H 4250 5050 50  0000 L CNN
+F 1 "22n" H 4250 5050 50  0000 L CNN
 F 2 "Capacitor_SMD:C_0805_2012Metric" H 4238 5000 50  0001 C CNN
 F 3 "~" H 4200 5150 50  0001 C CNN
@@
 P 4550 5150
 F 0 "C12" H 4665 5196 50  0000 L CNN
-F 1 "0.01u" H 4650 5050 50  0000 L CNN
+F 1 "22n" H 4650 5050 50  0000 L CNN
 F 2 "Capacitor_SMD:C_0805_2012Metric" H 4588 5000 50  0001 C CNN
 F 3 "~" H 4550 5150 50  0001 C CNN
@@
 P 1450 5150
 F 0 "C5" H 1565 5196 50  0000 L CNN
-F 1 "0.01u" H 1550 5050 50  0000 L CNN
+F 1 "22n" H 1550 5050 50  0000 L CNN
 F 2 "Capacitor_SMD:C_0805_2012Metric" H 1488 5000 50  0001 C CNN
 F 3 "~" H 1450 5150 50  0001 C CNN
@@
 P 1800 5150
 F 0 "C6" H 1915 5196 50  0000 L CNN
-F 1 "0.01u" H 1850 5050 50  0000 L CNN
+F 1 "22n" H 1850 5050 50  0000 L CNN
 F 2 "Capacitor_SMD:C_0805_2012Metric" H 1838 5000 50  0001 C CNN
 F 3 "~" H 1800 5150 50  0001 C CNN
@@
 P 14200 1300
 F 0 "C25" H 14400 1400 50  0000 C CNN
-F 1 "0.01u" H 14400 1300 50  0000 C CNN
+F 1 "10n" H 14400 1300 50  0000 C CNN
 F 2 "Capacitor_SMD:C_0805_2012Metric" H 14238 1150 50  0001 C CNN
 F 3 "~" H 14200 1300 50  0001 C CNN

Commit message: 0.47
backport from LrMAX coding and
Clean up LrE-6.2lpb old resources.
Other:
- note added: "F2.8-2"
- note removed: "F2.8-1"
Changed lines of the file:
@@
 	11650 1700 11650 1650
 Text Notes 14900 10450 0    197  ~ 0
-F2.8-1
+F2.8-2
 Wire Wire Line
 	1200 10900 1700 10900
